File: BaseCIAA7.sch (KiCad schematic (older format))
At the start: 8 parts, among them J10 Conn_02x12_Odd_Even, J13 Conn_02x05_Odd_Even, J18 Conn_02x05_Odd_Even, J6 Conn_02x12_Odd_Even

Commit message: version 3
Parts:
- added J9: Conn_02x12_Odd_Even, Connector_PinSocket_2.54mm:PinSocket_2x12_P2.54mm_Vertical, symbol Connector_Generic:Conn_02x12_Odd_Even
- added JX1: Conn_02x20_Counter_Clockwise, Poncho-PLC:TX24-40R-LT-H1E, symbol Connector_Generic:Conn_02x20_Counter_Clockwise
Connections:
- net labels added: ADC123_INP10, ADC12_INN1_INP0, ADC12_INN5_INP9, ADC12_INP15, ADC12_INP18, ADC12_INP19, ADC12_INP3, ADC12_INP5, ADC1_INP16, ADC3_INP1, PA15, PB3, PB4, PB5, PB6, PB7, PB8, PC10, PD3, PD4, PD5, PD6, PD7, PE2, PE3, PE4, PE5, PE6, ~RESET
- wire segments 64 -> 141
- no-connect marks 15 -> 11
Other:
- note added: "PONCHO CIAA7 EXPANSION CONNECTOR"
- moved on the sheet: H1, H2, H3, H4, J10, J13, J18, J6

Commit message: Version 4
Parts:
- added FID1, FID2, FID3: Fiducial, Fiducial:Fiducial_0.5mm_Mask1mm, symbol Mechanical:Fiducial
- added H5, H6, H7, H8: MountingHole, MountingHole:MountingHole_3.2mm_M3_Pad_Via, symbol Mechanical:MountingHole_Pad
- J8: renamed from JX1; Desc (none) -> 40 Position Connector Receptacle, Outer Shroud Contacts Thr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; Digikey# (none) -> 670-1386-ND
- renumbered J6 to J7
Connections:
- wire segments 141 -> 136
Other:
- note added: "CONECTOR DE EXPANSIÓN\n LATERAL\n"
- note added: "CONECTORES DE \nINTERCONEXION A CIAA7"
- note added: "SUJECIÓN Y\nFIDUCIALES\n"
- note removed: "CIAA7 EXPANSION CONNECTORS"
- note removed: "PONCHO CIAA7 EXPANSION CONNECTOR"
- moved on the sheet: H1, H2, H3, H4, J13, J18, J8

Commit message: Ruteo Parcial-Replanteo Esquematico pafa favorecer ruteo
Changed lines of the file:
@@
 Connection ~ 8950 5500
 Text HLabel 5400 4800 0    50   Input ~ 0
-IN0
+IN5
 Text HLabel 5400 4900 0    50   Input ~ 0
+IN3
+Text HLabel 5400 5000 0    50   Input ~ 0
 IN1
-Text HLabel 5400 5000 0    50   Input ~ 0
-IN2
 Text HLabel 10900 4600 2    50   Input ~ 0
 IN7
@@
 Wire Wire Line
 	5900 4400 5400 4400
-Text HLabel 5400 4400 0    50   Output ~ 0
+Text HLabel 6900 4700 2    50   Output ~ 0
 OUT0
-Text HLabel 5400 4500 0    50   Output ~ 0
+Text HLabel 6900 4600 2    50   Output ~ 0
 OUT1
 Text HLabel 5400 4600 0    50   Output ~ 0
@@
 Text HLabel 5400 4700 0    50   Output ~ 0
 OUT3
+Text HLabel 5400 4400 0    50   Output ~ 0
+OUT4
 Text HLabel 6900 4400 2    50   Output ~ 0
-OUT4
+OUT5
+Text HLabel 5400 4500 0    50   Output ~ 0
+OUT6
 Text HLabel 6900 4500 2    50   Output ~ 0
-OUT5
-Text HLabel 6900 4600 2    50   Output ~ 0
-OUT6
-Text HLabel 6900 4700 2    50   Output ~ 0
 OUT7
 Wire Wire Line
@@
 L power:+3.3V #PWR0150
 U 1 1 5DA49099
-P 1000 3450
-F 0 "#PWR0150" H 1000 3300 50  0001 C CNN
-F 1 "+3.3V" H 1015 3623 50  0000 C CNN
-F 2 "" H 1000 3450 50  0001 C CNN
-F 3 "" H 1000 3450 50  0001 C CNN
-	1    1000 3450
-	1    0    0    -1
-$EndComp
-$Comp
-L power:+5V #PWR0151
-U 1 1 5DA6E049
-P 1400 3150
-F 0 "#PWR0151" H 1400 3000 50  0001 C CNN
-F 1 "+5V" H 1415 3323 50  0000 C CNN
-F 2 "" H 1400 3150 50  0001 C CNN
-F 3 "" H 1400 3150 50  0001 C CNN
-	1    1400 3150
-	-1   0    0    -1
+P 1000 3700
+F 0 "#PWR0150" H 1000 3550 50  0001 C CNN
+F 1 "+3.3V" H 1015 3873 50  0000 C CNN
+F 2 "" H 1000 3700 50  0001 C CNN
+F 3 "" H 1000 3700 50  0001 C CNN
+	1    1000 3700
+	1    0    0    -1
 $EndComp
 Wire Wire Line
@@
 	6400 4800 6900 4800
 Text HLabel 6900 4800 2    50   Input ~ 0
-IN3
+IN4
 Text HLabel 6900 4900 2    50   Input ~ 0
-IN4
-Text HLabel 6900 5000 2    50   Input ~ 0
-IN5
+IN2
 Wire Wire Line
 	6400 5000 6900 5000
@@
 L power:GND #PWR01
 U 1 1 5DB34C57
-P 1250 3800
-F 0 "#PWR01" H 1250 3550 50  0001 C CNN
-F 1 "GND" H 1255 3627 50  0000 C CNN
-F 2 "" H 1250 3800 50  0001 C CNN
-F 3 "" H 1250 3800 50  0001 C CNN
-	1    1250 3800
-	1    0    0    -1
-$EndComp
-Wire Wire Line
-	1250 3700 1250 3800
+P 1250 4000
+F 0 "#PWR01" H 1250 3750 50  0001 C CNN
+F 1 "GND" H 1255 3827 50  0000 C CNN
+F 2 "" H 1250 4000 50  0001 C CNN
+F 3 "" H 1250 4000 50  0001 C CNN
+	1    1250 4000
+	1    0    0    -1
+$EndComp
+Wire Wire Line
+	1250 3700 1250 4000
 Wire Wire Line
 	2300 3700 1250 3700
-Wire Wire Line
-	2300 3800 1400 3800
-Wire Wire Line
-	1400 3800 1400 3150
 $Comp
 L power:+5V #PWR03
 U 1 1 5DB5877D
-P 3900 4150
-F 0 "#PWR03" H 3900 4000 50  0001 C CNN
-F 1 "+5V" H 3915 4323 50  0000 C CNN
-F 2 "" H 3900 4150 50  0001 C CNN
-F 3 "" H 3900 4150 50  0001 C CNN
-	1    3900 4150
+P 3900 3250
+F 0 "#PWR03" H 3900 3100 50  0001 C CNN
+F 1 "+5V" H 3915 3423 50  0000 C CNN
+F 2 "" H 3900 3250 50  0001 C CNN
+F 3 "" H 3900 3250 50  0001 C CNN
+	1    3900 3250
 	-1   0    0    -1
 $EndComp
@@
 	2800 5500 3900 5500
 Wire Wire Line
-	3900 5500 3900 4150
-$Comp
-L power:+3.3V #PWR02
-U 1 1 5DB6E070
-P 3750 4450
-F 0 "#PWR02" H 3750 4300 50  0001 C CNN
-F 1 "+3.3V" H 3765 4623 50  0000 C CNN
-F 2 "" H 3750 4450 50  0001 C CNN
-F 3 "" H 3750 4450 50  0001 C CNN
-	1    3750 4450
-	1    0    0    -1
-$EndComp
-Wire Wire Line
-	2800 4600 3750 4600
-Wire Wire Line
-	3750 4600 3750 4450
+	3900 5500 3900 4600
 Wire Wire Line
 	2300 4700 1000 4700
 Wire Wire Line
-	1000 4700 1000 3450
+	1000 4700 1000 3800
 $Comp
 L Mechanical:MountingHole_Pad H7
@@
 	1    0    0    -1
 $EndComp
+Connection ~ 1000 3800
+Wire Wire Line
+	1000 3800 2300 3800
+Wire Wire Line
+	2800 4600 3900 4600
+Connection ~ 3900 4600
+Wire Wire Line
+	3900 4600 3900 3250
+Wire Wire Line
+	1000 3700 1000 3800
+Text HLabel 6900 5000 2    50   Input ~ 0
+IN0
 $EndSCHEMATC
