File: BaseCIAA7.sch (KiCad schematic (older format))
At the start: 17 parts, among them J10 Conn_02x12_Odd_Even, J13 Conn_02x05_Odd_Even, J18 Conn_02x05_Odd_Even, J7 Conn_02x12_Odd_Even, J8 Conn_02x20_Counter_Clockwise, J9 Conn_02x12_Odd_Even

Commit message: Esq + PCB + Bom terminados
Parts:
- FID1, FID2, FID3: Desc (none) -> Fiducial
- H1, H2, H3, H4, H5, H6, H7, H8: Desc (none) -> Mounting Hole
- J10, J7: Desc (none) -> 2x12 Pin header - 2.54mm; Digikey# 2057-PH2-12-UA-ND -> 2057-PH2-12-UA-ND; DigikeyPage (none) -> https://www.digikey.com/products/en?keywords=2057-PH2-12-UA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; Manf (none) -> Adam
- J13, J18: Desc (none) -> 2x5 Pin header - 2.54mm; Digikey# 2057-PH2-12-UA-ND -> 2057-PH2-12-UA-ND; DigikeyPage (none) -> https://www.digikey.com/products/en?keywords=2057-PH2-12-UA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; Manf (none) -> Adam
- J8: Desc 40 Position Connector Receptacle, Outer Shroud Contacts Through Hole, Right Angle Gold -> 40 Position Connector Receptacle, Outer Shroud Contacts Through Hole, Right Angle Gold; Digikey# 670-1386-ND -> 670-1386-ND; DigikeyPage (none) -> https://www.digikey.com/products/en?keywords=670-1386-ND; Manf (none) -> Jae
- J9: Desc (none) -> 2x12 Pin header - 2.54mm; Digikey# (none) -> 2057-PH2-12-UA-ND; DigikeyPage (none) -> https://www.digikey.com/products/en?keywords=2057-PH2-12-UA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; Manf (none) -> Adam
Changed lines of the file:
@@
 F 2 "MountingHole:MountingHole_3.2mm_M3_Pad_Via" H 6850 750 50  0001 C CNN
 F 3 "~" H 6850 750 50  0001 C CNN
+F 4 "Mounting Hole" H 6850 750 50  0001 C CNN "Desc"
 	1    6850 750
 	0    -1   -1   0
@@
 F 2 "MountingHole:MountingHole_3.2mm_M3_Pad_Via" H 5150 750 50  0001 C CNN
 F 3 "~" H 5150 750 50  0001 C CNN
+F 4 "Mounting Hole" H 5150 750 50  0001 C CNN "Desc"
 	1    5150 750
 	0    1    -1   0
@@
 F 2 "MountingHole:MountingHole_3.2mm_M3_Pad_Via" H 4950 750 50  0001 C CNN
 F 3 "~" H 4950 750 50  0001 C CNN
+F 4 "Mounting Hole" H 4950 750 50  0001 C CNN "Desc"
 	1    4950 750
 	0    -1   1    0
@@
 F 1 "Conn_02x12_Odd_Even" H 9250 5400 50  0000 C CNN
 F 2 "Connector_PinSocket_2.54mm:PinSocket_2x12_P2.54mm_Vertical" H 8650 4700 50  0001 C CNN
-F 3 "" H 8650 4700 50  0001 C CNN
-F 4 " 	2057-PH2-12-UA-ND " H 8650 4700 50  0001 C CNN "Digikey#"
+F 3 "http://adam-tech.com/downloader.php?p=PH2-XX-UA.pdf" H 8650 4700 50  0001 C CNN
+F 4 "2057-PH2-12-UA-ND" H 8650 4700 50  0001 C CNN "Digikey#"
+F 5 "2x12 Pin header - 2.54mm" H 8650 4700 50  0001 C CNN "Desc"
+F 6 "Adam" H 8650 4700 50  0001 C CNN "Manf"
+F 7 "https://www.digikey.com/products/en?keywords=2057-PH2-12-UA-ND" H 8650 4700 50  0001 C CNN "DigikeyPage"
 	1    8650 4700
 	1    0    0    -1
@@
 F 1 "Conn_02x05_Odd_Even" H 8000 3050 50  0000 L CNN
 F 2 "Connector_PinSocket_2.54mm:PinSocket_2x05_P2.54mm_Vertical" H 8650 2700 50  0001 C CNN
-F 3 "PH2-XX-UA.pdf" H 8650 2700 50  0001 C CNN
-F 4 " 	2057-PH2-12-UA-ND " H 8650 2700 50  0001 C CNN "Digikey#"
+F 3 "http://adam-tech.com/downloader.php?p=PH2-XX-UA.pdf" H 8650 2700 50  0001 C CNN
+F 4 "2057-PH2-12-UA-ND" H 8650 2700 50  0001 C CNN "Digikey#"
+F 5 "2x5 Pin header - 2.54mm" H 8650 2700 50  0001 C CNN "Desc"
+F 6 "Adam" H 8650 2700 50  0001 C CNN "Manf"
+F 7 "https://www.digikey.com/products/en?keywords=2057-PH2-12-UA-ND" H 8650 2700 50  0001 C CNN "DigikeyPage"
 	1    8650 2700
 	-1   0    0    1
@@
 F 1 "Conn_02x05_Odd_Even" H 7700 3050 50  0000 C CNN
 F 2 "Connector_PinSocket_2.54mm:PinSocket_2x05_P2.54mm_Vertical" H 7350 2700 50  0001 C CNN
-F 3 "PH2-XX-UA.pdf" H 7350 2700 50  0001 C CNN
-F 4 " 	2057-PH2-12-UA-ND " H 7350 2700 50  0001 C CNN "Digikey#"
+F 3 "http://adam-tech.com/downloader.php?p=PH2-XX-UA.pdf" H 7350 2700 50  0001 C CNN
+F 4 "2057-PH2-12-UA-ND" H 7350 2700 50  0001 C CNN "Digikey#"
+F 5 "2x5 Pin header - 2.54mm" H 7350 2700 50  0001 C CNN "Desc"
+F 6 "Adam" H 7350 2700 50  0001 C CNN "Manf"
+F 7 "https://www.digikey.com/products/en?keywords=2057-PH2-12-UA-ND" H 7350 2700 50  0001 C CNN "DigikeyPage"
 	1    7350 2700
 	-1   0    0    1
@@
 F 1 "Conn_02x12_Odd_Even" H 10150 5326 50  0000 C CNN
 F 2 "Connector_PinSocket_2.54mm:PinSocket_2x12_P2.54mm_Vertical" H 10100 4700 50  0001 C CNN
-F 3 "" H 10100 4700 50  0001 C CNN
+F 3 "http://adam-tech.com/downloader.php?p=PH2-XX-UA.pdf" H 10100 4700 50  0001 C CNN
+F 4 "2x12 Pin header - 2.54mm" H 10100 4700 50  0001 C CNN "Desc"
+F 5 "2057-PH2-12-UA-ND" H 10100 4700 50  0001 C CNN "Digikey#"
+F 6 "Adam" H 10100 4700 50  0001 C CNN "Manf"
+F 7 "https://www.digikey.com/products/en?keywords=2057-PH2-12-UA-ND" H 10100 4700 50  0001 C CNN "DigikeyPage"
 	1    10100 4700
 	1    0    0    -1
@@
 F 2 "Poncho-PLC:TX24-40R-LT-H1E" H 2500 4600 50  0001 C CNN
 F 3 "https://www.jae.com/direct/topics/topics_file_download/?topics_id=66755&ext_no=06&index=0&_lang=en" H 2500 4600 50  0001 C CNN
-F 4 "	40 Position Connector Receptacle, Outer Shroud Contacts Through Hole, Right Angle Gold" H 2500 4600 50  0001 C CNN "Desc"
-F 5 "	670-1386-ND" H 2500 4600 50  0001 C CNN "Digikey#"
+F 4 "40 Position Connector Receptacle, Outer Shroud Contacts Through Hole, Right Angle Gold" H 2500 4600 50  0001 C CNN "Desc"
+F 5 "670-1386-ND" H 2500 4600 50  0001 C CNN "Digikey#"
+F 6 "Jae" H 2500 4600 50  0001 C CNN "Manf"
+F 7 "https://www.digikey.com/products/en?keywords=670-1386-ND" H 2500 4600 50  0001 C CNN "DigikeyPage"
 	1    2500 4600
 	1    0    0    -1
@@
 F 2 "MountingHole:MountingHole_3.2mm_M3_Pad_Via" H 7050 750 50  0001 C CNN
 F 3 "~" H 7050 750 50  0001 C CNN
+F 4 "Mounting Hole" H 7050 750 50  0001 C CNN "Desc"
 	1    7050 750
 	0    1    1    0
@@
 F 2 "MountingHole:MountingHole_3.2mm_M3_Pad_Via" H 5150 1050 50  0001 C CNN
 F 3 "~" H 5150 1050 50  0001 C CNN
+F 4 "Mounting Hole" H 5150 1050 50  0001 C CNN "Desc"
 	1    5150 1050
 	0    1    -1   0
@@
 F 2 "MountingHole:MountingHole_3.2mm_M3_Pad_Via" H 4950 1050 50  0001 C CNN
 F 3 "~" H 4950 1050 50  0001 C CNN
+F 4 "Mounting Hole" H 4950 1050 50  0001 C CNN "Desc"
 	1    4950 1050
 	0    -1   1    0
@@
 F 2 "Fiducial:Fiducial_0.5mm_Mask1mm" H 9700 950 50  0001 C CNN
 F 3 "~" H 9700 950 50  0001 C CNN
+F 4 "Fiducial" H 9700 950 50  0001 C CNN "Desc"
 	1    9700 950
 	1    0    0    -1
@@
 F 2 "Fiducial:Fiducial_0.5mm_Mask1mm" H 9100 950 50  0001 C CNN
 F 3 "~" H 9100 950 50  0001 C CNN
+F 4 "Fiducial" H 9100 950 50  0001 C CNN "Desc"
 	1    9100 950
 	1    0    0    -1
@@
 F 2 "Fiducial:Fiducial_0.5mm_Mask1mm" H 9400 950 50  0001 C CNN
 F 3 "~" H 9400 950 50  0001 C CNN
+F 4 "Fiducial" H 9400 950 50  0001 C CNN "Desc"
 	1    9400 950
 	1    0    0    -1
@@
 F 2 "MountingHole:MountingHole_3.2mm_M3_Pad_Via" H 7050 1050 50  0001 C CNN
 F 3 "~" H 7050 1050 50  0001 C CNN
+F 4 "Mounting Hole" H 7050 1050 50  0001 C CNN "Desc"
 	1    7050 1050
 	0    1    1    0
@@
 F 2 "MountingHole:MountingHole_3.2mm_M3_Pad_Via" H 6850 1050 50  0001 C CNN
 F 3 "~" H 6850 1050 50  0001 C CNN
+F 4 "Mounting Hole" H 6850 1050 50  0001 C CNN "Desc"
 	1    6850 1050
 	0    -1   -1   0
@@
 F 1 "Conn_02x12_Odd_Even" H 6700 5450 50  0000 C CNN
 F 2 "Connector_PinSocket_2.54mm:PinSocket_2x12_P2.54mm_Vertical" H 6200 4800 50  0001 C CNN
-F 3 "" H 6200 4800 50  0001 C CNN
-F 4 " 	2057-PH2-12-UA-ND " H 6200 4800 50  0001 C CNN "Digikey#"
+F 3 "http://adam-tech.com/downloader.php?p=PH2-XX-UA.pdf" H 6200 4800 50  0001 C CNN
+F 4 "2057-PH2-12-UA-ND" H 6200 4800 50  0001 C CNN "Digikey#"
+F 5 "2x12 Pin header - 2.54mm" H 6200 4800 50  0001 C CNN "Desc"
+F 6 "Adam" H 6200 4800 50  0001 C CNN "Manf"
+F 7 "https://www.digikey.com/products/en?keywords=2057-PH2-12-UA-ND" H 6200 4800 50  0001 C CNN "DigikeyPage"
 	1    6200 4800
 	-1   0    0    1
