File: Salidas.sch (KiCad schematic (older format))
At the start: 58 parts, among them J1 TB_1X2, J2 TB_1X3-PonchoPLC-rescue, J3 TB_1X2, J4 TB_1X2, J5 TB_1X2, J7 TB_1X2, Q1 FQT13N06L, Q2 FQT13N06L, Q3 FQT13N06L, Q4 FQT13N06L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

Commit message: version 3
Parts:
- J1, J3, J4, J5, J7: footprint TerminalBlock_Phoenix:TerminalBlock_Phoenix_MKDS-1,5-2_1x02_P5.00mm_Horizontal -> Poncho-PLC:TerminalBlock_4Ucon_1x02_P3.50mm_Horizontal
- J2: footprint TerminalBlock_Phoenix:TerminalBlock_Phoenix_MKDS-1,5-3_1x03_P5.00mm_Horizontal -> Poncho-PLC:TerminalBlock_4Ucon_1x03_P3.50mm_Horizontal
- renumbered D2 to D1, D3 to D2, D4 to D3, D1 to D4
Connections:
- wire segments 199 -> 203

Commit message: Version 4
Parts:
- removed J3, J4, J5, J7: TB_1X2, Poncho-PLC:TerminalBlock_4Ucon_1x02_P3.50mm_Horizontal, symbol Poncho-PLC7-rescue:TB_1X2-PonchoPLC-rescue
- added J3, J4, J5, J6: TB_1X2, Poncho-PLC:TerminalBlock_WECO_120-M-311_1x02_P5.00mm_Plug-in_PCB, symbol Poncho-PLC7-rescue:TB_1X2
- C1, C2, C3, C4: symbol Poncho-PLC7-rescue:C_MINI-PonchoPLC-rescue -> Poncho-PLC7-rescue:C_MINI; Desc (none) -> 0.1µF ±10% 50V Ceramic Capacitor X7R 1206 (3216 Metric); Digikey# 1276-1007-2-ND -> CL31B104KBCNNNL-ND
- C5, C6, C7, C8: symbol Poncho-PLC7-rescue:C_MINI-PonchoPLC-rescue -> Poncho-PLC7-rescue:C_MINI; Desc (none) -> 0.1µF -20%, +80% 50V Ceramic Capacitor Y5V (F) 0805 (2012 M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; Digikey# CL31B104KBCNNNL-ND -> 1276-1007-2-ND
- D1, D2, D3, D4, D5, D6, D7, D8: footprint LED_SMD:LED_0603_1608Metric -> LED_SMD:LED_0805_2012Metric; symbol Poncho-PLC7-rescue:LED-PonchoPLC-rescue -> Poncho-PLC7-rescue:LED; Desc led rojo smd 0603 -> Red LED Indication - Discrete 2.1V 0603 (1608 Metric)
- J1: value TB_1X2 -> TB_1X2-PonchoPLC-rescue; footprint Poncho-PLC:TerminalBlock_4Ucon_1x02_P3.50mm_Horizontal -> Poncho-PLC:TerminalBlock_WECO_120-M-311_1x02_P5.00mm_Plug-in_PCB; symbol Poncho-PLC7-rescue:TB_1X2-PonchoPLC-rescue -> Poncho-PLC7-rescue:TB_1X2
- J2: footprint Poncho-PLC:TerminalBlock_4Ucon_1x03_P3.50mm_Horizontal -> Poncho-PLC:TerminalBlock_WECO_120-M-311_1x03_P5.00mm_Plug-in_PCB; symbol Poncho-PLC7-rescue:TB_1X3-PonchoPLC-rescue -> Poncho-PLC7-rescue:TB_1X3
- JP1, JP2, JP3, JP4: symbol Poncho-PLC7-rescue:Jumper-PonchoPLC-rescue -> Poncho-PLC7-rescue:Jumper; Desc (none) -> Connector Header Through Hole
- Q1, Q2, Q3, Q4: symbol Poncho-PLC7-rescue:FQT13N06L-PonchoPLC-rescue -> Poncho-PLC7-rescue:FQT13N06L; Desc (none) -> N-Channel 60V 2.8A (Tc) 2.1W (Tc) Surface Mount SOT-223-4
- R1, R2, R3, R4: value 100k -> 100K; symbol Poncho-PLC7-rescue:R-PonchoPLC-rescue -> Poncho-PLC7-rescue:R; Desc (none) -> 1/8W Chip Resistor 0805; Digikey# CR0805-JW-103ELFTR-ND -> CR0805-JW-104ELFTR-ND
- R10, R11, R12, R13, R14, R15, R16, R5, R6, R7, R8, R9: symbol Poncho-PLC7-rescue:R-PonchoPLC-rescue -> Poncho-PLC7-rescue:R; Desc (none) -> 1/8W Chip Resistor 0805; Digikey# (none) -> CR0805-JW-331ELFTR-ND
- TH1, TH2, TH3, TH4: symbol Poncho-PLC7-rescue:THERMISTOR-PonchoPLC-rescue -> Poncho-PLC7-rescue:THERMISTOR; Desc (none) -> Polymeric PTC Resettable Fuse 6V 1A Ih Surface Mount 1206 (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
- U1, U2, U3, U4: symbol Poncho-PLC7-rescue:MCP1416-PonchoPLC-rescue -> Poncho-PLC7-rescue:MCP1416; Desc (none) -> Low-Side Gate Driver IC Non-Inverting SOT-23-5
- U5, U6, U7, U8: symbol CIAA_ACC:SSR -> Poncho-PLC7-rescue:SSR; Desc RELAY SSR SPST-NO 2A 60V 6SMD -> Solid State SPST-NO (1 Form A) 6-SMD (0.300\", 7.62mm)
Other:
- note added: "NOTA: SI SE OPTA POR MANEJAR\nLOS TRANSISTORES DIRECTAMENTE\nSIN MONTAR LOS DRIVER MCP1416\nES NECESARIO PUENTEAR LOS\nJUMPER JP1 AL JP4\nCASO CONTRARIO DEJARLOS\nABIERTOS"
- note added: "SALIDAS DIGITALES CON \nRELES DE ESTADO SÓLIDO"
- note added: "SALIDAS DIGITALES OPEN DRAIN"
- note removed: "ISOLATED DIGITAL OUTPUTS\nWITH SOLID STATE RELAYS"
- note removed: "OPEN DRAIN DIGITAL OUTPUTS"
