File: Salidas.sch (KiCad schematic (older format))
At the start: 58 parts, among them J1 TB_1X2-PonchoPLC-rescue, J2 TB_1X3-PonchoPLC-rescue, J3 TB_1X2, J4 TB_1X2, J5 TB_1X2, J6 TB_1X2, Q1 FQT13N06L, Q2 FQT13N06L, Q3 FQT13N06L, Q4 FQT13N06L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

Commit message: Esq + PCB + Bom terminados
Parts:
- C1, C2, C3, C4: DigikeyPage (none) -> https://www.digikey.com/products/en?keywords=CL31B104KBCNNN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; Manf (none) -> Samsung
- C5, C6, C7, C8: DigikeyPage (none) -> https://www.digikey.com/products/en?keywords=1276-1007-2-ND; Manf (none) -> Samsung
- D1, D2, D3, D4, D5, D6, D7, D8: DigikeyPage (none) -> https://www.digikey.com/products/en?keywords=1080-1583-2-ND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; Manf (none) -> Everlight
- J1: Desc (none) -> Terminal Block - Header, Male Pins, Shrouded -5mm -2 pos; Digikey# (none) -> A98062-ND; DigikeyPage (none) -> https://www.digikey.com/products/en?keywords=A98062-ND%20; Manf (none) -> Weco
- J2: Desc (none) -> Terminal Block - Header, Male Pins, Shrouded -5mm -3 pos; Digikey# (none) -> A98063-ND; DigikeyPage (none) -> https://www.digikey.com/products/en?keywords=A98063-ND; Manf (none) -> Weco
- J3, J4, J5, J6: value TB_1X2 -> TB_1X3-PonchoPLC-rescue; Desc (none) -> Terminal Block - Header, Male Pins, Shrouded -5mm -3 pos; Digikey# (none) -> A98063-ND; DigikeyPage (none) -> https://www.digikey.com/products/en?keywords=A98063-ND; Manf (none) -> Weco
- JP1, JP2, JP3, JP4: Digikey# 2057-PH2-12-UA-ND -> 2057-PH2-12-UA-ND; DigikeyPage (none) -> https://www.digikey.com/products/en?keywords=2057-PH2-12-UA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; Manf (none) -> Adam
- Q1, Q2, Q3, Q4: DigikeyPage (none) -> https://www.digikey.com/products/en?keywords=%20FQT13N06LTF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; Manf (none) -> Bourns
- R1, R2, R3, R4: DigikeyPage (none) -> https://www.digikey.com/products/en?keywords=CR0805-JW-104E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; Manf (none) -> Bourns
- R10, R11, R12, R13, R14, R15, R16, R5, R6, R7, R8, R9: Digikey# CR0805-JW-331ELFTR-ND -> CR0805-JW-331ELFTR-ND; DigikeyPage (none) -> https://www.digikey.com/products/en?keywords=CR0805-JW-331E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; Manf (none) -> Bourns
- TH1, TH2, TH3, TH4: DigikeyPage (none) -> https://www.digikey.com/products/en?keywords=%20283-3142-1-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; Manf (none) -> Cooper
- U1, U2, U3, U4: DigikeyPage (none) -> https://www.digikey.com/products/en?keywords=MCP1416T-E%2FO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; Manf (none) -> Microchip
- U5, U6, U7, U8: DigikeyPage (none) -> https://www.digikey.com/products/en?keywords=VO14642AABCT-ND; Manf# VO14642AABTR -> (none)

Commit message: Agregado Leds Entradas
Changed lines of the file:
@@
 F 1 "330" H 7790 2770 40  0000 C CNN
 F 2 "Resistor_SMD:R_0805_2012Metric" V 7830 2750 30  0001 C CNN
-F 3 "https://www.bourns.com/docs/Product-Datasheets/CHPREZTR.pdf" H 7900 2750 30  0000 C CNN
+F 3 "https://www.bourns.com/docs/Product-Datasheets/CHPREZTR.pdf" H 7900 2750 30  0001 C CNN
 F 4 "" H 7900 2750 60  0001 C CNN "Title"
 F 5 "1/8W Chip Resistor 0805 " H 7900 2750 50  0001 C CNN "Desc"
@@
 F 1 "330" H 7790 3770 40  0000 C CNN
 F 2 "Resistor_SMD:R_0805_2012Metric" V 7830 3750 30  0001 C CNN
-F 3 "https://www.bourns.com/docs/Product-Datasheets/CHPREZTR.pdf" H 7900 3750 30  0000 C CNN
+F 3 "https://www.bourns.com/docs/Product-Datasheets/CHPREZTR.pdf" H 7900 3750 30  0001 C CNN
 F 4 "" H 7900 3750 60  0001 C CNN "Title"
 F 5 "1/8W Chip Resistor 0805 " H 7900 3750 50  0001 C CNN "Desc"
