File: Entradas.sch (KiCad schematic (older format))
At the start: 22 parts, among them U9 SI8380P-IU

Commit message: Ruteo Casi terminado (faltan planos de masa)
Connections:
- net GND renamed GNDS
Changed lines of the file:
@@
-	1    0    0    -1
-$EndComp
-$Comp
-L power:GND #PWR0112
-U 1 1 5E027D09
-P 9050 3050
-F 0 "#PWR0112" H 9050 2800 50  0001 C CNN
-F 1 "GND" H 9055 2877 50  0000 C CNN
-F 2 "" H 9050 3050 50  0001 C CNN
-F 3 "" H 9050 3050 50  0001 C CNN
-	1    9050 3050
 	1    0    0    -1
 $EndComp
@@
 Text Label 6300 4400 0    50   ~ 0
 A8
+$Comp
+L power:GNDS #PWR?
+U 1 1 5DCA33B5
+P 9050 3050
+AR Path="/5DAD5FB7/5DCA33B5" Ref="#PWR?"  Part="1"
+AR Path="/5D8546B3/5DCA33B5" Ref="#PWR0112"  Part="1"
+F 0 "#PWR0112" H 9050 2800 50  0001 C CNN
+F 1 "GNDS" H 9150 2900 50  0000 R CNN
+F 2 "" H 9050 3050 50  0001 C CNN
+F 3 "" H 9050 3050 50  0001 C CNN
+	1    9050 3050
+	1    0    0    -1
+$EndComp
 $EndSCHEMATC
